Commit message: repostion_lidar

File: src/av_robot/urdf/robot.xacro (robot description, xacro)
@@ -30,5 +30,5 @@
     </joint>
     <joint name="hokuyo_joint" type="fixed">
-        <origin xyz="0.15 0 0.1" rpy="0 0 0"/>
+        <origin xyz="0.35 0 0.1" rpy="0 0 0"/>
         <parent link="chassis"/>
         <child link="hokuyo"/>
